File: GRIT_main/GRIT_main.kicad_sch (KiCad schematic)
At the start: 29 parts, among them J1 Raspberry_Pi_4, M1 Drive Motor Left, M2 Drive Motor Right, M3 Rotating Drum, M4 Flywheel, Q1 IRLZ34N, U1 Raspberry_Pi_Pico

Commit message: Updated Schematic
Parts:
- removed Motor_Driver_1, Motor_Driver_2, Motor_Driver_3, Motor_Driver_4: ~, symbol Custom_Symbols:12V_Motor_Controller
- added Dual_Motor_Driver: ~, symbol Custom_Symbols:12V_Dual_Motor_Driver
- added M5, M6: Fan, symbol Motor:Fan
- added Q2, Q3: Power Mosfet, Package_TO_SOT_SMD:PQFN_8x8, symbol Transistor_FET:FDMT80060DC
Connections:
- net at GPS.3 (GND), IMU.18 (GND), J1.14 (GND)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: now also Dual_Motor_Driver.3 (GND_a), Dual_Motor_Driver.4 (GND_b)
- net at Buck_Converter. (4), U1.48 (USB_VDD), US1.4 (Vcc)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: now also M6.1 (+)
- net at Buck_Converter. (4), F1.1, Q1.2 (D): now also Dual_Motor_Driver.16 (PWR+), Q2.3 (D), Q3.3 (D)
- net at D1.2 (A), Q1.3 (S): now also J1.12 (GPIO18/SPI1_~{CE0}/PCM_CLK/PWM0), Dual_Motor_Driver.7 (IN1_b)
- net at GPS.1 (Vcc), J1.2 (5V), J1.4 (5V)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: now also Dual_Motor_Driver.1 (Vcc_a), Dual_Motor_Driver.10 (EN_b), Dual_Motor_Driver.2 (Vcc_b), Dual_Motor_Driver.9 (EN_a)
- net at M3.2 (-): now also BT1.2 (-), Buck_Converter. (4), D2.1 (K), M4.2 (-), Dual_Motor_Driver.15 (PWR-)
- net at M3.1 (+): now also Q2.2 (S)
- net at J1.31 (GPCLK2/GPIO06): now also Q2.1 (G)
- net at Buck_Converter. (4): now also M6.2 (-)
- net at M4.1 (+): now also Q3.2 (S)
- net at J1.29 (GPCLK1/GPIO05): now also Q3.1 (G)
- net at J1.32 (GPIO12/PWM0): now also Dual_Motor_Driver.5 (IN1_a)
- net at J1.33 (GPIO13/PWM1): now also Dual_Motor_Driver.6 (IN2_a)
- net at J1.38 (GPIO20/SPI1_MOSI/PCM_DIN/PWM1): now also Dual_Motor_Driver.8 (IN2_b)
- net at M2.1 (+): now also Dual_Motor_Driver.14 (OUT_b+)
- net at M2.2 (-): now also Dual_Motor_Driver.13 (OUT_b-)
- net at M1.1 (+): now also Dual_Motor_Driver.18 (OUT_a+)
- net at M1.2 (-): now also Dual_Motor_Driver.17 (OUT_a-)
Other:
- moved on the sheet: BT1, F1, M1, M2, M3

Commit message: Final Schematic
Parts:
- removed Buck_Converter: ~, symbol Custom_Symbols:Buck_Converter_12V_to_5V
- removed Dual_Motor_Driver: ~, symbol Custom_Symbols:12V_Dual_Motor_Driver
- removed J1: Raspberry_Pi_4, symbol Connector:Raspberry_Pi_4
- removed LCD: ~, symbol Custom_Symbols:I2C_LCD_Screen
- removed LimitSwitch: ~, symbol Switch:SW_SPDT_XKB_DMx-xxxx-1
- removed M6: Fan, symbol Motor:Fan
- removed U1: Raspberry_Pi_Pico, Package_DFN_QFN:QFN-56-1EP_7x7mm_P0.4mm_EP3.2x3.2mm, symbol MCU_RaspberryPi:RP2040
- added BMS: INA260, Package_SO:TSSOP-16_4.4x5mm_P0.65mm, symbol Sensor:INA260
- added Buck_Converter1: ~, symbol Custom_Symbols:Buck_Converter_12V_to_5V
- added Dual_Motor_Driver1: ~, symbol Custom_Symbols:12V_Dual_Motor_Driver
- added LCD1: ~, symbol Custom_Symbols:I2C_LCD_Screen
- added LimitSwitch1: ~, symbol Switch:SW_SPDT_XKB_DMx-xxxx-1
- added M7: Onboard Fan, symbol Motor:Fan
- added R3, R4: 4.7k, symbol Device:R_US
- added Raspberry_Pi_Pico: ~, symbol Custom_Symbols:Custom_Raspberry_Pi_Pico
- added SW1, SW2: RotaryEncoder_Switch, symbol Device:RotaryEncoder_Switch
- added SW3, SW4, SW5, SW6: SW_Push_LED, symbol Switch:SW_Push_LED
- added SW7: E-Stop, Button_Switch_SMD:Nidec_Copal_CAS-120A, symbol Switch:SW_Nidec_CAS-120A1
- added SW8: Power Switch, Button_Switch_SMD:Nidec_Copal_CAS-120A, symbol Switch:SW_Nidec_CAS-120A1
- added U3: ~, symbol Custom_Symbols:Custom_Raspberry_Pi
- M5: value Fan -> Cooling Fan
Connections:
- net at US1.1 (Trig): now also Raspberry_Pi_Pico.4 (GPIO2)
- net at US1.2 (Echo): now also Raspberry_Pi_Pico.5 (GPIO3)
- net at US1.3 (GND), US2.3 (GND), US3.3 (GND)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: now also Raspberry_Pi_Pico.57 (GND); no longer GPS.3 (GND), IMU.18 (GND)
- net at US1.4 (Vcc), US2.4 (Vcc), US3.4 (Vcc)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: now also Raspberry_Pi_Pico.45 (VDD_REG)
- net at IMU.12 (INT): now also U3.7 (GPCLK0/GPIO04)
- net at IMU.13 (VDD), IMU.8 (VLOGIC): now also R1.2, R2.2, R3.2, R4.2, SW1.C, SW2.C, U3.1 (3V3), U3.17 (3V3); no longer R1.1, R2.1
- net at IMU.23 (SCL): now also U3.3 (SDA_I2C1/GPIO02)
- net at IMU.9 (AD0): now also U3.5 (SCL_I2C1/GPIO03)
- net at Q1.1 (G): now also U3.36 (GPIO16/SPI1_~{CE2})
- net at Q1.2 (D), Q2.3 (D), Q3.3 (D): now also Buck_Converter1. (4), Dual_Motor_Driver1.16 (PWR+), SW8.1 (C); no longer F1.1
- net at BT1.2 (-), D2.1 (K), M3.2 (-)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: now also BMS.11 (GND), BMS.6 (GND), Buck_Converter1. (4), Dual_Motor_Driver1.15 (PWR-)
- net at GPS.4 (Tx): now also U3.8 (GPIO14/UART_TXD)
- net at GPS.1 (Vcc): now also M5.1 (+), BMS.10 (VS), Dual_Motor_Driver1.1 (Vcc_a), Dual_Motor_Driver1.10 (EN_b), Dual_Motor_Driver1.2 (Vcc_b), Dual_Motor_Driver1.9 (EN_a), LCD1.1 (Vcc), SW1.A, SW2.A, SW3.4 (A), SW4.4 (A), SW5.4 (A), SW6.4 (A), U3.2 (5V), U3.4 (5V)
- net at Q3.1 (G): now also U3.35 (GPIO19/SPI1_MISO/PCM_FS)
- net at Q2.1 (G): now also U3.11 (GPIO17/SPI1_~{CE1})
- net at GPS.2 (GND): now also IMU.18 (GND), M5.2 (-), Dual_Motor_Driver1.3 (GND_a), Dual_Motor_Driver1.4 (GND_b), LCD1.3 (GND), LimitSwitch1.1 (A), SW1.B, SW2.B, SW3.2, SW4.2, SW5.2, SW6.2, U3.14 (GND), U3.20 (GND), U3.25 (GND), U3.30 (GND), U3.34 (GND), U3.39 (GND), U3.6 (GND), U3.9 (GND)
- net at M2.2 (-): now also Dual_Motor_Driver1.13 (OUT_b-)
- net at M2.1 (+): now also Dual_Motor_Driver1.14 (OUT_b+)
- net at M1.2 (-): now also Dual_Motor_Driver1.17 (OUT_a-)
- net at M1.1 (+): now also Dual_Motor_Driver1.18 (OUT_a+)
- net at US6.1 (Trig): now also Raspberry_Pi_Pico.15 (GPIO12)
- net at US6.2 (Echo): now also Raspberry_Pi_Pico.16 (GPIO13)
- net at US2.1 (Trig): now also Raspberry_Pi_Pico.6 (GPIO4)
- net at US2.2 (Echo): now also Raspberry_Pi_Pico.7 (GPIO5)
- net at US7.1 (Trig): now also Raspberry_Pi_Pico.17 (GPIO14)
- net at US7.2 (Echo): now also Raspberry_Pi_Pico.18 (GPIO15)
- net at BT1.1 (+), F1.2: now also BMS.12 (VBUS)
- net at US4.1 (Trig): now also Raspberry_Pi_Pico.11 (GPIO8)
- net at US4.2 (Echo): now also Raspberry_Pi_Pico.12 (GPIO9)
- net at US3.1 (Trig): now also Raspberry_Pi_Pico.8 (GPIO6)
- net at US3.2 (Echo): now also Raspberry_Pi_Pico.9 (GPIO7)
- net at US5.1 (Trig): now also Raspberry_Pi_Pico.13 (GPIO10)
- net at US5.2 (Echo): now also Raspberry_Pi_Pico.14 (GPIO11)
- new net: LCD1.2 (SCL), R2.1, U3.19 (MOSI_SPI0/GPIO10)
- new net: SW4.1, SW4.3 (K), U3.28 (ID_SC_I2C0/GPIO01)
- new net: BMS.1 (IN+), BMS.2 (IN+), BMS.3 (IN+)
- new net: BMS.14 (IN-), BMS.15 (IN-), BMS.16 (IN-)
- new net: BMS.8 (SDA), U3.37 (GPIO26/SDIO_DAT2)
- new net: BMS.9 (SCL), U3.22 (GPIO25/SDIO_DAT1)
- new net: F1.1, SW7.2 (B)
- new net: SW7.3 (A), SW8.2 (B)
- new net: SW6.1, SW6.3 (K), U3.26 (~{CE1}_SPI0/GPIO07)
- new net: LimitSwitch1.3 (C), U3.13 (GPIO27/SDIO_DAT3)
- new net: Buck_Converter1. (4), Raspberry_Pi_Pico. (USB_VDD), U3. (Vdd) (x2)
- new net: M7.1 (+), U3. (Vdd)
- new net: M7.2 (-), U3. (Vdd)
- new net: GPS.3 (Rx), U3.10 (GPIO15/UART_RXD)
- new net: Dual_Motor_Driver1.7 (IN1_b), U3.12 (GPIO18/SPI1_~{CE0}/PCM_CLK/PWM0)
- new net: SW2.S2, U3.15 (GPIO22/SDIO_CLK)
- new net: SW1.S1, U3.16 (GPIO23/SDIO_CMD)
- new net: SW1.S2, U3.18 (GPIO24/SDIO_DAT0)
- new net: R4.1, Raspberry_Pi_Pico.28 (GPIO17), U3.21 (MISO_SPI0/GPIO09)
- new net: LCD1.4 (SDA), R1.1, U3.23 (SCLK_SPI0/GPIO11)
- new net: R3.1, Raspberry_Pi_Pico.27 (GPIO16), U3.24 (~{CE0}_SPI0/GPIO08)
- new net: SW3.1, SW3.3 (K), U3.27 (ID_SD_I2C0/GPIO00)
- new net: SW5.1, SW5.3 (K), U3.29 (GPCLK1/GPIO05)
- new net: Dual_Motor_Driver1.5 (IN1_a), U3.32 (GPIO12/PWM0)
- new net: Dual_Motor_Driver1.6 (IN2_a), U3.33 (GPIO13/PWM1)
- new net: Dual_Motor_Driver1.8 (IN2_b), U3.38 (GPIO20/SPI1_MOSI/PCM_DIN/PWM1)
- new net: SW2.S1, U3.40 (GPIO21/SPI1_SCLK/PCM_DOUT)
Other:
- moved on the sheet: D1, D2, IMU, Q1

Commit message: Minor Fix
Parts:
- added R5, R6: 4.7k, symbol Device:R_US
Connections:
- net at IMU.13 (VDD), IMU.8 (VLOGIC), R1.2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: now also R5.2, R6.2
- net at BMS.8 (SDA), U3.37 (GPIO26/SDIO_DAT2): now also R5.1
- net at BMS.9 (SCL), U3.22 (GPIO25/SDIO_DAT1): now also R6.1
- new net: Buck_Converter1. (4), Raspberry_Pi_Pico. (USB_VDD), U3. (Vdd)
Changed lines of the file:
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@@
 	)
 	(junction
+		(at 251.46 104.14)
+		(diameter 0)
+		(color 0 0 0 0)
+	)
+	(junction
 		(at 154.94 53.34)
 		(diameter 0)
@@
 	)
 	(junction
+		(at 165.1 104.14)
+		(diameter 0)
+		(color 0 0 0 0)
+	)
+	(junction
 		(at 322.58 144.78)
 		(diameter 0)
@@
 	)
 	(junction
+		(at 162.56 162.56)
+		(diameter 0)
+		(color 0 0 0 0)
+	)
+	(junction
 		(at 127 177.8)
 		(diameter 0)
@@
 		(color 0 0 0 0)
 	)
+	(junction
+		(at 165.1 165.1)
+		(diameter 0)
+		(color 0 0 0 0)
+	)
 	(wire
 		(pts
@@
 	(wire
 		(pts
+			(xy 165.1 104.14) (xy 165.1 106.68)
+		)
+		(stroke
+			(width 0)
+			(type default)
+		)
+	)
+	(wire
+		(pts
 			(xy 120.65 50.8) (xy 157.48 50.8)
 		)
@@
 	(wire
 		(pts
+			(xy 165.1 104.14) (xy 162.56 104.14)
+		)
+		(stroke
+			(width 0)
+			(type default)
+		)
+	)
+	(wire
+		(pts
 			(xy 110.49 177.8) (xy 110.49 140.97)
 		)
@@
 	(wire
 		(pts
+			(xy 162.56 114.3) (xy 162.56 162.56)
+		)
+		(stroke
+			(width 0)
+			(type default)
+		)
+	)
+	(wire
+		(pts
 			(xy 182.88 147.32) (xy 54.61 147.32)
 		)
@@
 	(wire
 		(pts
+			(xy 165.1 114.3) (xy 165.1 165.1)
+		)
+		(stroke
+			(width 0)
+			(type default)
+		)
+	)
+	(wire
+		(pts
 			(xy 41.91 275.59) (xy 41.91 35.56)
 		)
@@
 	(wire
 		(pts
+			(xy 251.46 104.14) (xy 165.1 104.14)
+		)
+		(stroke
+			(width 0)
+			(type default)
+		)
+	)
+	(wire
+		(pts
 			(xy 59.69 124.46) (xy 59.69 245.11)
 		)
@@
 	(wire
 		(pts
-			(xy 251.46 124.46) (xy 251.46 53.34)
+			(xy 251.46 124.46) (xy 251.46 104.14)
 		)
 		(stroke
@@
 	(wire
 		(pts
+			(xy 162.56 104.14) (xy 162.56 106.68)
+		)
+		(stroke
+			(width 0)
+			(type default)
+		)
+	)
+	(wire
+		(pts
 			(xy 148.59 74.93) (xy 148.59 160.02)
 		)
@@
 	(wire
 		(pts
+			(xy 251.46 104.14) (xy 251.46 53.34)
+		)
+		(stroke
+			(width 0)
+			(type default)
+		)
+	)
+	(wire
+		(pts
 			(xy 180.34 243.84) (xy 180.34 246.38)
 		)
@@
 	)
 	(symbol
+		(lib_id "Device:R_US")
+		(at 165.1 110.49 180)
+		(unit 1)
+		(exclude_from_sim no)
+		(in_bom yes)
+		(on_board yes)
+		(dnp no)
+		(property "Reference" "R5"
+			(at 166.37 109.22 0)
+			(effects
+				(font
+					(size 1.27 1.27)
+				)
+				(justify right)
+			)
+		)
+		(property "Value" "4.7k"
+			(at 166.37 111.76 0)
+			(effects
+				(font
+					(size 1.27 1.27)
+				)
+				(justify right)
+			)
+		)
+		(property "Footprint" ""
+			(at 164.084 110.236 90)
+			(effects
+				(font
+					(size 1.27 1.27)
+				)
+				(hide yes)
+			)
+		)
+		(property "Datasheet" "~"
+			(at 165.1 110.49 0)
+			(effects
+				(font
+					(size 1.27 1.27)
+				)
+				(hide yes)
+			)
+		)
+		(property "Description" "Resistor, US symbol"
+			(at 165.1 110.49 0)
+			(effects
+				(font
+					(size 1.27 1.27)
+				)
+				(hide yes)
+			)
+		)
+		(pin "1"
+		)
+		(pin "2"
+		)
+		(instances
+			(project "GRIT_main"
+				(path "/8d650bef-20d2-4446-89ff-47284d65b67c"
+					(reference "R5")
+					(unit 1)
+				)
+			)
+		)
+	)
+	(symbol
 		(lib_id "Custom_Symbols:I2C_LCD_Screen")
 		(at 285.75 149.86 0)
@@
 					(unit 1)
 				)
+			)
+		)
+	)
+	(symbol
+		(lib_id "Device:R_US")
+		(at 162.56 110.49 0)
+		(mirror x)
+		(unit 1)
+		(exclude_from_sim no)
+		(in_bom yes)
+		(on_board yes)
+		(dnp no)
+		(property "Reference" "R6"
+			(at 161.29 109.22 0)
+			(effects
+				(font
+					(size 1.27 1.27)
+				)
+				(justify right)
+			)
+		)
+		(property "Value" "4.7k"
+			(at 161.29 111.76 0)
+			(effects
+				(font
+					(size 1.27 1.27)
+				)
+				(justify right)
+			)
+		)
+		(property "Footprint" ""
+			(at 163.576 110.236 90)
+			(effects
+				(font
+					(size 1.27 1.27)
+				)
+				(hide yes)
+			)
+		)
+		(property "Datasheet" "~"
+			(at 162.56 110.49 0)
+			(effects
+				(font
+					(size 1.27 1.27)
+				)
+				(hide yes)
+			)
+		)
+		(property "Description" "Resistor, US symbol"
+			(at 162.56 110.49 0)
+			(effects
+				(font
+					(size 1.27 1.27)
+				)
+				(hide yes)
+			)
+		)
+		(pin "1"
+		)
+		(pin "2"
+		)
+		(instances
+			(project "GRIT_main"
+				(path "/8d650bef-20d2-4446-89ff-47284d65b67c"
+					(reference "R6")
+					(unit 1)
+				)
