File: GRIT_main_pcb/GRIT_main_pcb.kicad_pcb (KiCad board)
At the start: 4 copper layers, 80 x 80 mm, 37 parts

Commit message: 1st layer done
Parts:
- removed HMI: HMI Connection, Connector_PinHeader_2.54mm:PinHeader_1x02_P2.54mm_Vertical
- added 10k: PB 1 Pull Down, Resistor_THT:R_Axial_DIN0207_L6.3mm_D2.5mm_P5.08mm_Vertical, F.Cu at (40.5, 84.2)
- added LCD: LCD Screen, Connector_PinHeader_2.54mm:PinHeader_1x04_P2.54mm_Vertical, F.Cu at (74.0, 24.5)
- added LED+: LED+, Connector_PinHeader_2.54mm:PinHeader_1x01_P2.54mm_Vertical, F.Cu at (89.8, 55.2)
- added LED-: LED-, Connector_PinHeader_2.54mm:PinHeader_1x01_P2.54mm_Vertical, F.Cu at (89.0, 89.0)
- GPS: moved to B.Cu
- PowMOS1: renamed from Power MOS 1
- PowMOS2: renamed from Power MOS 2
- Raspberry Pi: moved to B.Cu
- Rel1: renamed from Relay 1
- Rel2: renamed from Relay 2
- moved PowMOS1 66.7 mm to (33.8, 73.5), turned to 90 degrees
- moved PowMOS2 55.9 mm to (47.0, 82.5)
- moved GPS 46.4 mm to (62.0, 60.5), turned to -90 degrees
- moved Limit Switch 42.8 mm to (35.2, 79.9)
- moved 4.7k 36.0 mm to (66.8, 83.6)
- moved 4.7k 36.0 mm to (73.2, 83.6)
- moved BMS 36.0 mm to (60.6, 87.9)
- moved EncL 35.8 mm to (26.7, 58.5)
- moved EncR 27.3 mm to (52.7, 58.5)
- moved IMU 15.8 mm to (17.0, 80.8), turned to 180 degrees
- moved 10k 15.0 mm to (30.4, 33.5)
- moved EStop 14.5 mm to (30.5, 16.7)
- moved Raspberry Pi 14.4 mm to (74.8, 69.3), turned to 90 degrees
- moved 4.7k 14.1 mm to (37.8, 51.8)
- moved Pico 13.5 mm to (20.9, 48.0)
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- renumbered On/Off to On
Connections:
- 10k pad 1: (no net) -> 5V (x5)
- 10k pad 2: (no net) -> PI28
- 10k pad 2: (no net) -> On
- 10k pad 2: (no net) -> PI29
- 10k pad 2: (no net) -> PI26
- 10k pad 2: (no net) -> EStop
- 4.7k pad 1: (no net) -> PI22
- 4.7k pad 2: (no net) -> 3V3 (x4)
- 4.7k pad 1: (no net) -> PI24
- 4.7k pad 1: (no net) -> PI37
- 4.7k pad 1: (no net) -> 3V3 (x2)
- 4.7k pad 2: (no net) -> PI23
- 4.7k pad 1: (no net) -> PI21
- 4.7k pad 2: (no net) -> PI19
- BMS pad 1: (no net) -> 5V
- BMS pad 2: (no net) -> GND
- BMS pad 3: (no net) -> PI22
- BMS pad 4: (no net) -> PI37
- Cooling Fan pad 1: (no net) -> GND
- Cooling Fan pad 2: (no net) -> 5V
- Dual Motor Driver pad 1: (no net) -> 5V
- Dual Motor Driver pad 10: (no net) -> 5V
- Dual Motor Driver pad 2: (no net) -> 5V
- Dual Motor Driver pad 3: (no net) -> GND
- Dual Motor Driver pad 4: (no net) -> GND
- Dual Motor Driver pad 5: (no net) -> PI32
- Dual Motor Driver pad 6: (no net) -> PI12
- Dual Motor Driver pad 7: (no net) -> PI33
- Dual Motor Driver pad 8: (no net) -> PI38
- Dual Motor Driver pad 9: (no net) -> 5V
- EStop pad 1: (no net) -> GND
- EStop pad 2: (no net) -> EStop
- EncL pad 1: (no net) -> 3V3
- EncL pad 10: (no net) -> GND
- EncL pad 2: (no net) -> 5V
- EncL pad 5: (no net) -> PI15
- EncL pad 7: (no net) -> PI40
- EncR pad 1: (no net) -> 3V3
- EncR pad 10: (no net) -> GND
- EncR pad 2: (no net) -> 5V
- EncR pad 5: (no net) -> PI18
- EncR pad 7: (no net) -> PI16
- GPS pad 1: (no net) -> 5V
- GPS pad 2: (no net) -> PI10
- GPS pad 3: (no net) -> PI8
- GPS pad 4: (no net) -> GND
- IMU pad 1: (no net) -> 3V3
- IMU pad 2: (no net) -> GND
- IMU pad 3: (no net) -> PI3
- IMU pad 4: (no net) -> PI5
- IMU pad 8: (no net) -> PI7
- LED1 pad 1: (no net) -> LED1
- LED1 pad 2: (no net) -> LED2
- LED1 pad 1: (no net) -> LED2
- LED1 pad 2: (no net) -> LED-
- LED3 pad 1: (no net) -> LED3
- LED3 pad 2: (no net) -> LED4
- LED4 pad 1: (no net) -> LED4
- LED4 pad 2: (no net) -> LED-
- Limit Switch pad 1: (no net) -> PI13
- Limit Switch pad 2: (no net) -> 5V
- MOS1 pad 1: (no net) -> PI36
- MOS1 pad 2: (no net) -> LED+
- MOS1 pad 3: (no net) -> LED3
- MOS2 pad 1: (no net) -> PI31
- MOS2 pad 2: (no net) -> LED+
- MOS2 pad 3: (no net) -> LED1
- On pad 1: (no net) -> GND
- On pad 2: (no net) -> On
- PB 1 pad 1: (no net) -> GND
- PB 1 pad 2: (no net) -> PI26
- PB 2 pad 1: (no net) -> GND
- PB 2 pad 2: (no net) -> PI28
- PB 3 pad 1: (no net) -> GND
- PB 3 pad 2: (no net) -> PI29
- Pico pad 1: (no net) -> PI21
- Pico pad 2: (no net) -> PI24
- PowMOS1 pad 1: (no net) -> PI35
- PowMOS1 pad 2: (no net) -> GND
- PowMOS2 pad 1: (no net) -> PI11
- PowMOS2 pad 2: (no net) -> GND
- Raspberry Pi pad 1: (no net) -> 3V3
- Raspberry Pi pad 10: (no net) -> PI10
- Raspberry Pi pad 11: (no net) -> PI11
- Raspberry Pi pad 12: (no net) -> PI12
- Raspberry Pi pad 13: (no net) -> PI13
- Raspberry Pi pad 14: (no net) -> GND
- Raspberry Pi pad 15: (no net) -> PI15
- Raspberry Pi pad 16: (no net) -> PI16
- Raspberry Pi pad 17: (no net) -> 3V3
- Raspberry Pi pad 18: (no net) -> PI18
- Raspberry Pi pad 19: (no net) -> PI19
- Raspberry Pi pad 2: (no net) -> 5V
- Raspberry Pi pad 20: (no net) -> GND
- Raspberry Pi pad 21: (no net) -> PI21
- Raspberry Pi pad 22: (no net) -> PI22
- Raspberry Pi pad 23: (no net) -> PI23
- Raspberry Pi pad 24: (no net) -> PI24
- Raspberry Pi pad 25: (no net) -> GND
- Raspberry Pi pad 26: (no net) -> PI26
- Raspberry Pi pad 27: (no net) -> PI27
- Raspberry Pi pad 28: (no net) -> PI28
- Raspberry Pi pad 29: (no net) -> PI29
- Raspberry Pi pad 3: (no net) -> PI3
- Raspberry Pi pad 30: (no net) -> GND
- Raspberry Pi pad 31: (no net) -> PI31
- Raspberry Pi pad 32: (no net) -> PI32
- Raspberry Pi pad 33: (no net) -> PI33
- Raspberry Pi pad 34: (no net) -> GND
- Raspberry Pi pad 35: (no net) -> PI35
- Raspberry Pi pad 36: (no net) -> PI36
- Raspberry Pi pad 37: (no net) -> PI37
- Raspberry Pi pad 38: (no net) -> PI38
- Raspberry Pi pad 39: (no net) -> GND
- Raspberry Pi pad 4: (no net) -> 5V
- Raspberry Pi pad 40: (no net) -> PI40
- Raspberry Pi pad 5: (no net) -> PI5
- Raspberry Pi pad 6: (no net) -> GND
- Raspberry Pi pad 7: (no net) -> PI7
- Raspberry Pi pad 8: (no net) -> PI8
- Raspberry Pi pad 9: (no net) -> GND
- Rel1 pad 1: (no net) -> EStop
- Rel2 pad 1: (no net) -> On
Routing:
- net (no net): track 249.6 -> 0.00 mm
- net GND: track 0.00 -> 199.7 mm
- net 3V3: track 0.00 -> 185.7 mm
- net 5V: track 0.00 -> 128.7 mm
- net PI7: track 0.00 -> 72.9 mm
- net PI3: track 0.00 -> 70.2 mm
- net PI5: track 0.00 -> 67.6 mm
- net PI15: track 0.00 -> 54.4 mm
- net PI24: track 0.00 -> 36.1 mm
- net PI13: track 0.00 -> 28.7 mm
- net PI11: track 0.00 -> 20.6 mm
- net LED+: track 0.00 -> 17.2 mm
- net EStop: track 0.00 -> 15.0 mm
- net LED-: track 0.00 -> 14.2 mm
- net PI23: track 0.00 -> 11.1 mm
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
Commit message: Final Main PCB
Parts:
- added REF**: MountingHole_2.5mm, MountingHole:MountingHole_2.5mm, F.Cu at (16.5, 87.5)
- added REF**: MountingHole_2.5mm, MountingHole:MountingHole_2.5mm, F.Cu at (87.5, 16.5)
- moved 4.7k 4.14 mm to (41.9, 51.8)
- moved Dual Motor Driver 3.50 mm to (79.7, 34.8)
Connections:
- 10k pad 2: PI28 -> PI26
- 10k pad 2: PI26 -> PI28
- PB 1 pad 2: PI26 -> PI28
- PB 2 pad 2: PI28 -> PI26
- Raspberry Pi pad 14: GND -> (no net)
- Raspberry Pi pad 17: 3V3 -> (no net)
- Raspberry Pi pad 20: GND -> (no net)
- Raspberry Pi pad 25: GND -> (no net)
- Raspberry Pi pad 30: GND -> (no net)
- Raspberry Pi pad 34: GND -> (no net)
- Raspberry Pi pad 6: GND -> (no net)
- Raspberry Pi pad 9: GND -> (no net)
Routing:
- net GND: track 199.7 -> 0.00 mm
- net PI21: track 9.53 -> 166.8 mm
- net PI23: track 11.1 -> 160.6 mm
- net PI36: track 0.00 -> 142.9 mm
- net 5V: track 128.7 -> 269.0 mm
- net PI29: track 4.94 -> 133.4 mm
- net PI33: track 0.00 -> 106.7 mm
- net PI19: track 9.89 -> 104.7 mm
- net PI32: track 0.00 -> 87.8 mm
- net PI38: track 0.00 -> 76.4 mm
- net PI31: track 0.00 -> 65.4 mm
- net PI37: track 7.81 -> 72.8 mm
- net PI22: track 4.80 -> 64.0 mm
- net PI28: track 4.94 -> 48.3 mm
- net PI12: track 0.00 -> 43.3 mm
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- added copper zone on In2.Cu, net GND

Commit message: Sub PCB Updated
Parts:
- Rel1, Rel2: value Relay Control -> PinHeader_1x03_P2.54mm_Vertical; footprint Connector_PinHeader_2.54mm:PinHeader_1x01_P2.54mm_Vertical -> Connector_PinHeader_2.54mm:PinHeader_1x03_P2.54mm_Vertical
- moved Rel2 2.80 mm to (35.0, 21.0)
- moved Rel1 2.28 mm to (25.0, 17.0)
Connections:
- Raspberry Pi pad 4: 5V -> (no net)
- Rel1 pad 1: EStop -> GND
- Rel2 pad 1: On -> GND
Routing:
- net 5V: track 269.0 -> 285.4 mm
