File: GRIT_main_sub_PCB/GRIT_main_sub_PCB.kicad_pcb (KiCad board)
At the start: 4 copper layers, 9 parts

Commit message: 1st layer done
Parts:
- removed the REF** at (106.8, 59.0)
- added REF**: PinHeader_1x20_P2.54mm_Vertical, Connector_PinHeader_2.54mm:PinHeader_1x20_P2.54mm_Vertical, F.Cu at (55.8, 22.9)
- added REF**: PinHeader_1x20_P2.54mm_Vertical, Connector_PinHeader_2.54mm:PinHeader_1x20_P2.54mm_Vertical, F.Cu at (38.1, 22.9)
- moved Vdd 60.1 mm to (19.6, 24.9)
- moved Vdd 60.1 mm to (19.6, 62.9)
- moved Vdd 60.1 mm to (28.1, 62.9)
- moved Vdd 60.1 mm to (19.6, 37.6)
- moved Vdd 60.1 mm to (28.1, 37.6)
- moved Vdd 60.1 mm to (28.1, 24.9)
- moved Vdd 60.1 mm to (19.6, 50.2)
- moved Vdd 60.1 mm to (28.1, 50.2)
- renumbered REF** to Vdd
Routing:
- net (no net): track 1005.2 -> 1012.8 mm
Other:
- board outline added: 58.4 x 71.1 mm

Commit message: Sub PCB Updated
Parts:
- added REF**: MountingHole_2.5mm, MountingHole:MountingHole_2.5mm, F.Cu at (16.2, 16.8)
- added REF**: MountingHole_2.5mm, MountingHole:MountingHole_2.5mm, F.Cu at (16.2, 79.0)
- added REF**: MountingHole_2.5mm, MountingHole:MountingHole_2.5mm, F.Cu at (60.5, 16.8)
- added REF**: MountingHole_2.5mm, MountingHole:MountingHole_2.5mm, F.Cu at (60.5, 79.0)
- Pico 1: renamed from REF**
- Pico 40: renamed from REF**
- moved Vdd 1.52 mm to (18.8, 23.6)
- moved Vdd 1.52 mm to (27.2, 23.6)
- moved Vdd 1.50 mm to (18.8, 64.1)
- moved Vdd 1.50 mm to (27.2, 64.1)
- moved Vdd 1.46 mm to (27.3, 48.9)
- moved Vdd 1.40 mm to (18.8, 49.0)
- moved Pico 1 1.00 mm to (37.2, 23.4)
- moved Pico 40 1.00 mm to (55.0, 23.4)
- moved Vdd 0.95 mm to (18.8, 37.1)
- moved Vdd 0.93 mm to (27.3, 37.1)
Connections:
- Pico 1 pad 1: (no net) -> GP0
- Pico 1 pad 10: (no net) -> GP7
- Pico 1 pad 11: (no net) -> GP8
- Pico 1 pad 12: (no net) -> GP9
- Pico 1 pad 14: (no net) -> GP10
- Pico 1 pad 15: (no net) -> GP11
- Pico 1 pad 16: (no net) -> GP12
- Pico 1 pad 17: (no net) -> GP13
- Pico 1 pad 19: (no net) -> GP14
- Pico 1 pad 2: (no net) -> GP1
- Pico 1 pad 20: (no net) -> GP15
- Pico 1 pad 4: (no net) -> GP2
- Pico 1 pad 5: (no net) -> GP3
- Pico 1 pad 6: (no net) -> GP4
- Pico 1 pad 7: (no net) -> GP5
- Pico 1 pad 9: (no net) -> GP6
- Pico 40 pad 1: (no net) -> 5V
- Pico 40 pad 3: (no net) -> GND
- Vdd pad 1: (no net) -> 5V (x8)
- Vdd pad 2: (no net) -> GP0
- Vdd pad 3: (no net) -> GP1
- Vdd pad 4: (no net) -> GND (x8)
- Vdd pad 2: (no net) -> GP14
- Vdd pad 3: (no net) -> GP15
- Vdd pad 2: (no net) -> GP12
- Vdd pad 3: (no net) -> GP13
- Vdd pad 2: (no net) -> GP4
- Vdd pad 3: (no net) -> GP5
- Vdd pad 2: (no net) -> GP6
- Vdd pad 3: (no net) -> GP7
- Vdd pad 2: (no net) -> GP2
- Vdd pad 3: (no net) -> GP3
- Vdd pad 2: (no net) -> GP10
- Vdd pad 3: (no net) -> GP11
- Vdd pad 2: (no net) -> GP8
- Vdd pad 3: (no net) -> GP9
Routing:
- net (no net): track 1012.8 -> 0.00 mm
- net GP1: track 0.00 -> 29.0 mm
- net GP0: track 0.00 -> 27.4 mm
- net GP5: track 0.00 -> 26.2 mm
- net GP14: track 0.00 -> 26.0 mm
- net GP4: track 0.00 -> 24.7 mm
- net GP15: track 0.00 -> 24.3 mm
- net GP10: track 0.00 -> 23.9 mm
- net GP11: track 0.00 -> 23.0 mm
- net GP13: track 0.00 -> 12.1 mm
- net GP12: track 0.00 -> 12.1 mm
- net GP3: track 0.00 -> 12.0 mm
- net GP2: track 0.00 -> 12.0 mm
- net GP7: track 0.00 -> 11.6 mm
- net GP6: track 0.00 -> 11.6 mm
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- added copper zone on In1.Cu, net 5V
- added copper zone on In2.Cu, net GND
Other:
- board size 58.4 x 71.1 mm -> 52.9 x 72.1 mm
